File: pcb/sd.kicad_pcb (KiCad board)
At the start: 2 copper layers, 30.5 x 24.1 mm, 8 parts, among them J1 Micro_SD_Card_Det2, J2 Conn_01x09

Commit message: Ready for order
Routing:
- net GND: vias 14 -> 39
Other:
- board text added: "(MISO) DO"
- board text added: "(MOSI) DI"
- board text added: "CS"
- board text added: "SCLK"
- board text added: "SPI:"

Commit message: Bumped work revision to b.  Added capacitors which may or may not be needed.
Parts:
- added C1: 10uF, Capacitor_SMD:C_0603_1608Metric, F.Cu at (153.7, 85.1)
- added C2: 100nF, Capacitor_SMD:C_0603_1608Metric, F.Cu at (155.6, 85.1)
- moved R1 1.91 mm to (153.7, 90.2)
- moved R2 1.91 mm to (155.6, 90.2)
- moved R3 1.91 mm to (157.5, 90.2)
Routing:
- net VCC: track 46.9 -> 54.0 mm
- net /D3: track 33.7 -> 34.8 mm
- net /DET: track 20.9 -> 21.8 mm
- net /D2: track 32.0 -> 32.7 mm
- net GND: vias 39 -> 40
Other:
- board text added: "SPI"
- board text removed: "SPI:"

Commit message: More tweaks
Routing:
- net VCC: track 54.0 -> 49.5 mm
- net GND: vias 40 -> 44
Changed lines of the file:
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@@
+	)
+	(via
+		(at 173.99 90.805)
+		(size 0.7)
+		(drill 0.35)
+		(layers "F.Cu" "B.Cu")
+		(free yes)
+		(net 1)
 	)
 	(via
@@
 	)
 	(via
+		(at 173.99 93.345)
+		(size 0.7)
+		(drill 0.35)
+		(layers "F.Cu" "B.Cu")
+		(free yes)
+		(net 1)
+	)
+	(via
 		(at 156.845 84.8964)
 		(size 0.7)
@@
 	)
 	(via
+		(at 165.1 90.17)
+		(size 0.7)
+		(drill 0.35)
+		(layers "F.Cu" "B.Cu")
+		(free yes)
+		(net 1)
+	)
+	(via
 		(at 150.495 93.98)
 		(size 0.7)
@@
 	)
 	(via
-		(at 162.56 92.075)
+		(at 163.83 92.075)
 		(size 0.7)
 		(drill 0.35)
@@
 	)
 	(via
+		(at 173.99 100.965)
+		(size 0.7)
+		(drill 0.35)
+		(layers "F.Cu" "B.Cu")
+		(free yes)
+		(net 1)
+	)
+	(via
 		(at 160.02 99.06)
 		(size 0.7)
@@
 	)
 	(via
-		(at 173.99 96.52)
-		(size 0.7)
-		(drill 0.35)
-		(layers "F.Cu" "B.Cu")
-		(free yes)
-		(net 1)
-	)
-	(via
-		(at 168.275 95.25)
+		(at 173.99 95.885)
+		(size 0.7)
+		(drill 0.35)
+		(layers "F.Cu" "B.Cu")
+		(free yes)
+		(net 1)
+	)
+	(via
+		(at 168.91 91.44)
 		(size 0.7)
 		(drill 0.35)
@@
 		(free yes)
 		(net 1)
-	)
-	(segment
-		(start 172.72 88.265)
-		(end 159.385 88.265)
-		(width 0.4572)
-		(layer "F.Cu")
-		(net 2)
 	)
 	(segment
@@
 	)
 	(segment
+		(start 156.985 85.865)
+		(end 159.11 87.99)
+		(width 0.4572)
+		(layer "F.Cu")
+		(net 2)
+	)
+	(segment
 		(start 157.48 95.695)
 		(end 158.075 95.695)
@@
 	)
 	(segment
+		(start 167.48 90.645)
+		(end 167.48 94.53)
+		(width 0.4572)
+		(layer "F.Cu")
+		(net 2)
+	)
+	(segment
+		(start 155.575 85.865)
+		(end 156.985 85.865)
+		(width 0.4572)
+		(layer "F.Cu")
+		(net 2)
+	)
+	(segment
 		(start 158.075 95.695)
 		(end 158.56 95.21)
@@
 	)
 	(segment
+		(start 159.11 87.99)
+		(end 164.825 87.99)
+		(width 0.4572)
+		(layer "F.Cu")
+		(net 2)
+	)
+	(segment
+		(start 168.305 95.355)
+		(end 171.7575 95.355)
+		(width 0.4572)
+		(layer "F.Cu")
+		(net 2)
+	)
+	(segment
 		(start 158.56 89.66)
 		(end 158.245 89.345)
@@
 	)
 	(segment
-		(start 156.985 85.865)
-		(end 155.575 85.865)
-		(width 0.4572)
-		(layer "F.Cu")
-		(net 2)
-	)
-	(segment
 		(start 158.245 89.345)
 		(end 157.48 89.345)
@@
 	)
 	(segment
+		(start 167.48 94.53)
+		(end 168.305 95.355)
+		(width 0.4572)
+		(layer "F.Cu")
+		(net 2)
+	)
+	(segment
 		(start 155.575 89.345)
 		(end 157.48 89.345)
@@
 	)
 	(segment
-		(start 173.355 95.0897)
-		(end 173.355 88.9)
-		(width 0.4572)
-		(layer "F.Cu")
-		(net 2)
-	)
-	(segment
 		(start 155.575 95.695)
 		(end 157.48 95.695)
@@
 	)
 	(segment
-		(start 171.7575 95.355)
-		(end 173.0897 95.355)
-		(width 0.4572)
-		(layer "F.Cu")
-		(net 2)
-	)
-	(segment
-		(start 173.0897 95.355)
-		(end 173.355 95.0897)
+		(start 164.825 87.99)
+		(end 167.48 90.645)
 		(width 0.4572)
 		(layer "F.Cu")
@@
 	)
 	(segment
-		(start 159.385 88.265)
-		(end 156.985 85.865)
-		(width 0.4572)
-		(layer "F.Cu")
-		(net 2)
-	)
-	(segment
 		(start 150 85.865)
 		(end 149.225 85.09)
@@
 	)
 	(segment
-		(start 173.355 88.9)
-		(end 172.72 88.265)
-		(width 0.4572)
-		(layer "F.Cu")
-		(net 2)
-	)
-	(segment
 		(start 170.245 96.455)
 		(end 170.18 96.52)
@@
 		(net 6)
 	)
+	(via
+		(at 169.545 92.71)
+		(size 0.7)
+		(drill 0.35)
+		(layers "F.Cu" "B.Cu")
+		(net 6)
+	)
+	(segment
+		(start 164.85 91.92)
+		(end 163.1 90.17)
+		(width 0.2286)
+		(layer "B.Cu")
+		(net 6)
+	)
+	(segment
+		(start 163.1 90.17)
+		(end 147.955 90.17)
+		(width 0.2286)
+		(layer "B.Cu")
+		(net 6)
+	)
 	(segment
 		(start 169.545 92.71)
 		(end 168.91 92.71)
 		(width 0.2286)
-		(layer "F.Cu")
-		(net 6)
-	)
-	(via
-		(at 168.91 92.71)
-		(size 0.7)
-		(drill 0.35)
-		(layers "F.Cu" "B.Cu")
-		(net 6)
-	)
-	(segment
-		(start 164.05 91.92)
-		(end 164.045 91.925)
-		(width 0.2286)
-		(layer "B.Cu")
-		(net 6)
-	)
-	(segment
-		(start 162.29 90.17)
-		(end 147.955 90.17)
-		(width 0.2286)
 		(layer "B.Cu")
 		(net 6)
@@
 	(segment
 		(start 168.12 91.92)
-		(end 164.05 91.92)
-		(width 0.2286)
-		(layer "B.Cu")
-		(net 6)
-	)
-	(segment
-		(start 162.29 90.17)
-		(end 164.045 91.925)
+		(end 164.85 91.92)
 		(width 0.2286)
 		(layer "B.Cu")
@@
 	)
 	(segment
-		(start 168.55 94.255)
+		(start 170.31 94.255)
 		(end 171.7575 94.255)
 		(width 0.2286)
@@
 	)
 	(segment
-		(start 168.275 93.98)
-		(end 168.55 94.255)
+		(start 170.035 93.98)
+		(end 170.31 94.255)
+		(width 0.2286)
+		(layer "F.Cu")
+		(net 8)
+	)
+	(segment
+		(start 168.91 93.98)
+		(end 170.035 93.98)
 		(width 0.2286)
 		(layer "F.Cu")
@@
 	)
 	(via
-		(at 168.275 93.98)
+		(at 168.91 93.98)
 		(size 0.7)
 		(drill 0.35)
@@
 	)
 	(segment
+		(start 168.275 93.98)
+		(end 168.91 93.98)
+		(width 0.2286)
+		(layer "B.Cu")
+		(net 8)
+	)
+	(segment
 		(start 147.955 92.71)
 		(end 159.625 92.71)
@@
 	)
 	(segment
+		(start 170.18 91.44)
+		(end 170.795 92.055)
+		(width 0.2286)
+		(layer "F.Cu")
+		(net 9)
+	)
+	(segment
 		(start 152.845 90.17)
 		(end 153.67 90.995)
@@
 	)
 	(segment
-		(start 170.16 92.055)
-		(end 169.545 91.44)
+		(start 170.795 92.055)
+		(end 171.7575 92.055)
 		(width 0.2286)
 		(layer "F.Cu")
@@
 		(net 9)
 	)
-	(segment
-		(start 171.7575 92.055)
-		(end 170.16 92.055)
-		(width 0.2286)
-		(layer "F.Cu")
-		(net 9)
-	)
-	(via
-		(at 169.545 91.44)
-		(size 0.7)
-		(drill 0.35)
-		(layers "F.Cu" "B.Cu")
-		(net 9)
-	)
-	(segment
-		(start 165.36 90.77)
-		(end 162.22 87.63)
-		(width 0.2286)
-		(layer "B.Cu")
-		(net 9)
-	)
-	(segment
-		(start 169.51 91.44)
-		(end 168.84 90.77)
-		(width 0.2286)
-		(layer "B.Cu")
-		(net 9)
-	)
-	(segment
-		(start 168.84 90.77)
-		(end 165.36 90.77)
-		(width 0.2286)
-		(layer "B.Cu")
-		(net 9)
-	)
-	(segment
-		(start 169.545 91.44)
-		(end 169.51 91.44)
-		(width 0.2286)
-		(layer "B.Cu")
-		(net 9)
-	)
-	(segment
-		(start 162.22 87.63)
+	(via
+		(at 170.18 91.44)
+		(size 0.7)
+		(drill 0.35)
+		(layers "F.Cu" "B.Cu")
+		(net 9)
+	)
+	(segment
+		(start 169.51 90.77)
+		(end 167.005 90.77)
+		(width 0.2286)
+		(layer "B.Cu")
+		(net 9)
+	)
+	(segment
+		(start 167.005 90.77)
+		(end 163.865 87.63)
+		(width 0.2286)
+		(layer "B.Cu")
+		(net 9)
+	)
+	(segment
+		(start 170.18 91.44)
+		(end 169.51 90.77)
+		(width 0.2286)
+		(layer "B.Cu")
+		(net 9)
+	)
+	(segment
+		(start 163.865 87.63)
 		(end 147.955 87.63)
 		(width 0.2286)

Commit message: More tweaks
Routing:
- net /DET: track 21.8 -> 23.5 mm
- net /D1: track 32.9 -> 33.6 mm
- net GND: vias 44 -> 46
Changed lines of the file:
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@@
 	)
 	(gr_text "D2"
-		(at 149.86 87.63 0)
+		(at 149.225 87.63 0)
 		(layer "F.SilkS")
 		(effects
@@
 	)
 	(gr_text "D1"
-		(at 149.86 100.33 0)
+		(at 149.225 100.33 0)
 		(layer "F.SilkS")
 		(effects
@@
 	)
 	(gr_text "DET"
-		(at 149.86 102.87 0)
+		(at 149.225 102.87 0)
 		(layer "F.SilkS")
 		(effects
@@
 	)
 	(gr_text "CLK"
-		(at 149.86 95.25 0)
+		(at 149.225 95.25 0)
 		(layer "F.SilkS")
 		(effects
@@
 	)
 	(gr_text "D3"
-		(at 149.86 90.17 0)
+		(at 149.225 90.17 0)
 		(layer "F.SilkS")
 		(effects
@@
 	)
 	(gr_text "GND"
-		(at 149.86 105.41 0)
+		(at 149.225 105.41 0)
 		(layer "F.SilkS")
 		(effects
@@
 	)
 	(gr_text "CMD\n"
-		(at 149.86 92.71 0)
+		(at 149.225 92.71 0)
 		(layer "F.SilkS")
 		(effects
@@
 	)
 	(gr_text "VCC"
-		(at 149.86 85.09 0)
+		(at 149.225 85.09 0)
 		(layer "F.SilkS")
 		(effects
@@
 	)
 	(gr_text "D0"
-		(at 149.86 97.79 0)
+		(at 149.225 97.79 0)
 		(layer "F.SilkS")
 		(effects
@@
 	)
 	(via
-		(at 158.115 99.06)
+		(at 156.845 99.06)
 		(size 0.7)
 		(drill 0.35)
@@
 	)
 	(via
+		(at 159.385 91.44)
+		(size 0.7)
+		(drill 0.35)
+		(layers "F.Cu" "B.Cu")
+		(free yes)
+		(net 1)
+	)
+	(via
 		(at 173.99 100.965)
 		(size 0.7)
@@
 	)
 	(via
-		(at 160.02 99.06)
+		(at 159.385 99.06)
 		(size 0.7)
 		(drill 0.35)
@@
 	(via
 		(at 155.575 93.98)
+		(size 0.7)
+		(drill 0.35)
+		(layers "F.Cu" "B.Cu")
+		(free yes)
+		(net 1)
+	)
+	(via
+		(at 159.385 93.98)
 		(size 0.7)
 		(drill 0.35)
@@
 	)
 	(segment
-		(start 155.575 97.345)
-		(end 152.59 100.33)
+		(start 153.67 100.33)
+		(end 147.955 100.33)
 		(width 0.2286)
 		(layer "F.Cu")
@@
 	)
 	(segment
+		(start 155.575 98.425)
+		(end 153.67 100.33)
+		(width 0.2286)
+		(layer "F.Cu")
+		(net 4)
+	)
+	(segment
 		(start 171.7575 99.755)
 		(end 170.24 99.755)
@@
 	)
 	(segment
-		(start 152.59 100.33)
-		(end 147.955 100.33)
+		(start 155.575 97.345)
+		(end 155.575 98.425)
 		(width 0.2286)
 		(layer "F.Cu")
@@
 	)
 	(segment
+		(start 154.94 102.87)
+		(end 147.955 102.87)
+		(width 0.2286)
+		(layer "F.Cu")
+		(net 5)
+	)
+	(segment
 		(start 159.8425 94.9825)
 		(end 160.9575 93.8675)
@@
 	)
 	(segment
-		(start 147.955 102.87)
-		(end 151.955 102.87)
+		(start 157.48 97.345)
+		(end 157.48 100.33)
+		(width 0.2286)
+		(layer "F.Cu")
+		(net 5)
+	)
+	(segment
+		(start 157.48 100.33)
+		(end 154.94 102.87)
 		(width 0.2286)
 		(layer "F.Cu")
@@
 		(width 0.2286)
 		(layer "F.Cu")
-		(net 5)
-	)
-	(segment
-		(start 151.955 102.87)
-		(end 157.48 97.345)
-		(width 0.2286)
-		(layer "F.Cu")

Commit message: About to order
Other:
- board text added: "${TITLE} Rev. ${REVISION} ${COMPANY}"
- board text removed: "${TITLE} Rev. ${REVISION}"
Changed lines of the file:
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@@
 		)
 	)
-	(gr_text "${TITLE}\nRev. ${REVISION}"
-		(at 175.26 90.17 0)
+	(gr_text "${TITLE}\nRev. ${REVISION}\n${COMPANY}"
+		(at 175.895 87.63 0)
 		(layer "B.SilkS")
 		(effects
@@
 				(thickness 0.1)
 			)
-			(justify left bottom mirror)
+			(justify left top mirror)
 		)
 	)
